Commit message: Hoan thanh read_joint_stat

File: src/car/urdf/car.urdf (robot description, URDF)
Before this commit: robot car, 14 links, 13 joints
Joints:
- joint joint1: limit lower=-1.57 upper=1.57 effort=0 velocity=0 -> lower=-1.57 upper=1.52 effort=0 velocity=0
- joint joint_0: limit lower=-1.57 upper=3.14 effort=0 velocity=0 -> lower=-1.42 upper=3.14 effort=0 velocity=0
- joint joint_2: limit lower=-1.57 upper=1.57 effort=0 velocity=0 -> lower=-1.38 upper=1.726 effort=0 velocity=0
- joint joint_3: limit lower=-1.57 upper=1.57 effort=0 velocity=0 -> lower=-0.977 upper=2.13 effort=0 velocity=0
- joint joint_4: limit lower=-1.57 upper=1.57 effort=0 velocity=0 -> lower=-1.55 upper=1.55 effort=0 velocity=0

Commit message: Backup 24/05/2021: Adjusting navparam

File: src/car/urdf/car.urdf (robot description, URDF)
Before this commit: robot car, 15 links, 14 joints
Joints:
- joint dummy_joint: origin (none) -> xyz=0 0 0.11 rpy=0 0 0

Commit message: Backup 19/06/2021: Add them pi_camera de detect aruco

File: src/car/urdf/car.urdf (robot description, URDF)
Before this commit: robot car, 15 links, 14 joints
Joints:
- joint dummy_joint: origin xyz=0 0 0.11 rpy=0 0 0 -> (none)
- joint joint_5: limit lower=-0.01 upper=1.57 effort=0 velocity=0 -> lower=-3.14 upper=3.14 effort=0 velocity=0
