Commit message: Backup 25/06/2021: Execute arm to package on shelf

File: src/robot_description/urdf/robot_description.urdf (robot description, URDF)
Before this commit: robot robot_description, 16 links, 15 joints
Links:
- link base_link: mass 0.0416209175694483 -> 0.041621
- link link_1: mass 0.0798083268201474 -> 0.079808
- link link_2: mass 0.0475993853789399 -> 0.04759938537894
- link link_4: mass 0.0508687988735335 -> 0.0508687992629349
- link link_53: mass 0.00137328199751957 -> 0.00137328199751958
- link wh_bl: mass 0.0727548969777259 -> 0.0727548969777271
- link wh_br: mass 0.0727548969707371 -> 0.072755
- link wh_fl: mass 0.0727548969703373 -> 0.072755
Joints:
- joint joint_3: origin xyz=0.130508913511003 0 0 rpy=0.0330134851352869 0 0 -> xyz=0.13051 0 0 rpy=0.033013 0 0
- joint joint_4: axis 0.530861074931385 0.761296866307477 -0.372308474887572 -> 0.53086 0.7613 -0.37231; limit lower=-3.14 upper=0.3 effort=0 velocity=0 -> lower=-0.1 upper=0.1 effort=0 velocity=0; origin xyz=-0.0438541371732808 0.0759575937060697 0.0112859927951114 rpy=-0.116608909241159 -0.712230377732912 -1.84069508617415 -> xyz=-0.043854 0.075958 -0.008714 rpy=-0.11661 -0.71223 -1.8407; type continuous -> revolute
- joint joint_5: origin xyz=0.00617286993879481 -0.00952626535605935 0.0109219809266578 rpy=0.602136293756852 0.853540316865174 3.01057033246525 -> xyz=0.0061729 -0.0095263 0.010922 rpy=0.60214 0.85354 3.0106
- joint joint_51: origin xyz=-0.00360894860261653 0.0308388542215121 -0.00175000000000791 rpy=0 0 0 -> xyz=-0.0036089 0.030839 -0.00175 rpy=0 0 0
- joint joint_53: origin xyz=-0.0105213588774653 -0.00832612259373525 -0.0104276575228086 rpy=0.602136293756852 0.853540316865174 3.01057033246525 -> xyz=-0.0105213588774655 -0.00832612259373461 -0.0104276575228075 rpy=0.602136293756852 0.853540316865174 3.01057033246525
- joint joint_54: origin xyz=0.00344200446641575 0.0308579332581168 0 rpy=0 0 0 -> xyz=0.00344200446641575 0.0308579332581169 0 rpy=0 0 0
